File: electronics/holo/holo.brd (EAGLE design)
At the start: 164.8 x 150.7 mm, 98 parts, among them IC1 TP4056, IC2 TP4056, U1 CD4051BM, U2 CD4051BM, U4 CD4051BM

Commit message: Removing all components that will be replaced
Parts:
- removed BUT: KMR211GLFS, okie:PUSHBUTTON-KMR241GLFS
- removed C20, C21: 18pF, SparkFun-Passives:0805
- removed CA2, CA3: C_EU-100NF, rhoban:C0805
- removed D4, D5: Blue, SparkFun:LED-1206
- removed EXT: CONNEC_1X09, rhoban:CONNEC_1X09
- removed IC1, IC2: TP4056, TP4056:SOP-8
- removed OSC: 8MHz, SparkFun2:CRYSTAL-SMD-5X3
- removed P1, P2: (no value), jst-ph:JST-PH2
- removed PROGRAM: CONNEC_1X066PADS, rhoban:6PADS
- removed R10, R12, R24, R9: 5K, SparkFun-Passives:0805
- removed R11, R26, R30, R36, R46, R49: 1K, SparkFun-Passives:0805
- removed R18, R48: 10K, SparkFun-Passives:0805
- removed R25: 2K, SparkFun-Passives:0805
- removed R37, R38: 10K, rcl:R0805
- removed R47, R52: 4K, SparkFun-Passives:0805
- removed U$10, U$7: (no value), rhoban:430186070716
- removed U$18: NPN_BC817,215, rhoban:SOT-23
- removed U$24: LM2940IMP-5.0, rhoban:SOT223
- removed U$25: TS2940CW-3.3RP, rhoban:SOT223
- removed U$8: HOLO_OPTICALS, rhoban:HOLO_OPTICALS
- removed U2, U4: CD4051BM, rhoban:SOIC127P600X175-16N
- removed UC1: STM32F103CBT6, stm32:LQFP48
- added C13, C14, C9: (no value), rcl:153CLV-1010
- added C15, C16: 22uF, resistor:C0805
- added L1: IHLP2525CZER220M11IND_IHLP_2525_CZ_VIS-M, INDUCTOR:IND_IHLP_2525_CZ_VIS-M
- added MOS: SUD50N04-8M8P-4GE3, rhoban:TO252
- added R1: 270, rcl:R2010
- added R2: 2k, resistor:M0805
- added R4: 68k, resistor:M0805
- added R6: (no value), resistor:M0805
- added REG, REG1: REG_5V, rhoban:TRACOPOWER
- added X20: (no value), powersupply:DC-21MM
- C1, C2, C3, C4: value 10uF -> (none); device SparkFun-Passives:0805 -> rcl:153CLV-1010
- C12, C7: value 1uF -> (none); device SparkFun-Passives:0805 -> rcl:153CLV-1010
- D1: value Blue -> PMEG4030EP; device SparkFun:LED-1206 -> nxp_60:SOD128
- U$1: value GY-85 -> CONNEC_1X01PAD; device rhoban:GY-85 -> rhoban:1_PAD
- U$2, U$6: value (none) -> CONNEC_1X01PAD; device rhoban:430186070716 -> rhoban:1_PAD
- U$4: value HC05 -> CONNEC_1X01PAD; device rhoban:HC-05 -> rhoban:1_PAD
- U$5: value GP2 -> CONNEC_1X01PAD; device rhoban:GP2_THROUGH -> rhoban:1_PAD
- U1: value CD4051BM -> MT3608; device rhoban:SOIC127P600X175-16N -> MT3608:SOT95P280X145-6N
- moved U$4 221.4 mm to (-94.2, -194.6), turned to 0 degrees
- moved U$5 218.4 mm to (-89.9, -194.6), flipped to the top, turned to 0 degrees
- moved C4 217.2 mm to (-90.2, -154.8)
- moved U$6 202.2 mm to (-85.6, -194.6), turned to 0 degrees
- moved C1 191.9 mm to (-79.0, -130.8), turned to 0 degrees
- moved U$1 178.0 mm to (-54.0, -189.0), turned to 0 degrees
- moved C2 176.1 mm to (-66.7, -130.8)
- moved C3 171.4 mm to (-54.4, -130.8), turned to 0 degrees
- moved C12 165.5 mm to (-90.2, -167.4), turned to 0 degrees
- moved U1 163.9 mm to (-56.8, -164.6), turned to 0 degrees
- moved D1 160.5 mm to (-69.2, -188.7)
- moved U$2 159.2 mm to (-49.7, -189.0), turned to 0 degrees
- moved C7 127.8 mm to (-77.9, -154.8), turned to 0 degrees
Connections:
- removed net ADDR1: U1.11, U2.11, U4.11, UC1.38
- removed net ADDR2: U1.10, U2.10, U4.10, UC1.40
- removed net ADDR3: U1.9, U2.9, U4.9, UC1.14
- removed net A_INT: U$1.A_INT1
- removed net BOOT1: PROGRAM.4, UC1.20
- removed net BTN1: U$2.1, U$2.3, U2.1
- removed net BTN2: U$6.1, U$6.3, U4.1
- removed net BTN3: U$7.1, U$7.3, U1.5
- removed net BTN4: U$10.1, U$10.3, U2.5
- removed net BUTTON: BUT.P$2, BUT.P$4, R48.1, UC1.37, UC1.44
- removed net CHARGE_EN: IC1.8, IC2.8, R25.1
- removed net G_DRDY: U$1.M_DRDY
- removed net G_INT: U$1.G_INT
- removed net HAS_USB: R46.1, UC1.25
- removed net IMU_NC: U$1.VCC_IN
- removed net IMU_SCL: EXT.7, U$1.SCL, UC1.21
- removed net IMU_SDA: EXT.6, U$1.SDA, UC1.22
- removed net IN1: EXT.8, U2.4
- removed net IN2: EXT.9, U4.4
- removed net KEY: UC1.45
- removed net LED: R36.1, UC1.34
- removed net MORE_CHARGE: R47.1, R52.1, UC1.27
- removed net MRX: U$4.TX, UC1.13
- removed net MTX: U$4.RX, UC1.12
- removed net MUX1: U1.3, UC1.11
- removed net MUX2: U2.3, UC1.15
- removed net MUX3: U4.3, UC1.19
- removed net N$20: D4.A, R26.2
- removed net N$21: D5.C, IC2.7
- removed net N$22: IC2.6, R12.1
- removed net N$23: D5.A, R11.2
- removed net N$26: BUT.P$1, BUT.P$3, R49.2
- removed net N$29: D1.A, R36.2
- removed net N$33: R30.2, U$18.1
- removed net N$8: IC1.6, R10.1
- removed net OPTICAL1: U$8.O1, U1.15
- removed net OPTICAL2: U$8.O2, U2.15
- removed net OPTICAL3: U$8.O3, U4.15
- removed net OPTICAL4: U$8.O4, U1.12
- removed net OPTICAL5: U$8.O5, U2.12
- removed net OPTICAL6: U$8.O6, U4.12
- removed net OPTICAL7: U$8.O7, U1.1
- removed net OPTICAL_EN1: U$8.EN1, UC1.2
- removed net OPTICAL_EN2: U$8.EN2, UC1.3
- removed net OPTICAL_EN3: UC1.4
- removed net OSC_IN: C21.2, OSC.3, UC1.5
- removed net OSC_OUT: C20.2, OSC.1, UC1.6
- removed net P1: U$5.VO, U1.2
- removed net P2: U2.2
- removed net P3: U4.2
- removed net PROG1: IC1.2, R12.2, R24.2, R47.2
- removed net PROG2: IC2.2, R10.2, R52.2, R9.2
- removed net P_EN: R30.1, UC1.41
- removed net P_GND: U$18.3, U$5.GND
- removed net RX1: EXT.4, PROGRAM.6, R18.2, UC1.31
- removed net TX1: EXT.5, PROGRAM.5, UC1.30
- removed net VBAT: UC1.1
- removed net VOLTAGE1: R3.1, R5.2, U4.5
- removed net VOLTAGE2: R37.1, R38.2, U1.4
- removed net XBEECONF: U$4.KEY, UC1.39
- new net 1: X20.1
- new net 3.3V: REG1.P$3
- new net KICK: MOS.1, R6.1, U$4.1
- new net KICKER: MOS.3, U$6.1
- new net N$1: D1.2, L1.1, U1.1
- new net N$4: R2.2, R4.1, U1.3
- new net VOLTAGE: R3.1, R5.2
- new net VSTORE: C1.+, C12.+, C13.+, C14.+, C2.+, C3.+, C4.+, C7.+, C9.+, R1.1, U$5.1
- net 3.3: no longer C12.2, C7.2, CA3.1, EXT.2, PROGRAM.2, R49.1, U$1.3.3, U$25.3, U$4.3.3, U$8.3.3V, U1.16, U2.16, U4.16, UC1.24, UC1.36, UC1.48, UC1.9
- net BAT1+: no longer C3.2, IC1.5, P2.2
- net BAT2+: no longer P1.2
- net BAT2-: no longer C5.2, C6.2, C8.2, LED1.1-VDD, LED2.1-VDD, LED3.1-VDD, LED4.1-VDD, LED5.1-VDD, LED6.1-VDD, P1.1, R37.2, U$8.VIN
- net BAT2CHARGE: no longer C4.2, IC2.5
- net BUZZER: no longer UC1.10
- net DISC: no longer UC1.46
- net GND: now also C1.-, C12.-, C13.-, C14.-, C15.2, C16.2, C2.-, C3.-, C4.-, C7.-, C9.-, MOS.2, R2.1, R6.2, REG.P$2, REG1.P$2, U$1.1, U1.2, X20.3; no longer C1.1, C12.1, C2.1, C20.1, C21.1, C3.1, C4.1, C7.1, CA2.2, CA3.2, D1.C, EXT.1, IC1.1, IC1.3, IC2.1, IC2.3, P2.1, PROGRAM.1, R18.1, R24.1, R38.1, R48.2, R9.1, U$1.GND, U$10.2, U$10.4, U$18.2, U$2.2, U$2.4, U$24.2, U$24.4, U$25.2, U$4.GND, U$6.2, U$6.4, U$7.2, U$7.4, U$8.GND, U1.6, U1.7, U1.8, U2.6, U2.7, U2.8, U4.6, U4.7, U4.8, UC1.23, UC1.35, UC1.47, UC1.8
- net LEDS: no longer UC1.28
- net M1A: no longer UC1.43
- net M1B: no longer UC1.42
- net M1C1: no longer U1.13
- net M1C2: no longer U2.13
- net M2A: no longer UC1.16
- net M2B: no longer UC1.29
- net M2C1: no longer U4.13
- net M2C2: no longer U1.14
- net M3A: no longer UC1.18
- net M3B: no longer UC1.17
- net M3C1: no longer U2.14
- net M3C2: no longer U4.14
- net N$2: now also C16.1, D1.1, R1.2, R4.2; no longer D4.C, IC1.7
- net RESET: no longer PROGRAM.3, UC1.7
- net USBDM: no longer UC1.32
- net USBDP: no longer UC1.33
- net VCC: now also C5.2, C6.2, C8.2, LED1.1-VDD, LED2.1-VDD, LED3.1-VDD, LED4.1-VDD, LED5.1-VDD, LED6.1-VDD, REG.P$3; no longer CA2.1, U$24.3, U$25.1, U$5.VCC
- net VIN: now also C15.1, L1.2, REG.P$1, REG1.P$1, U$2.1, U1.4, U1.5, X20.2; no longer U$24.1
- net VIN_RAW: no longer EXT.3
- net VUSB: no longer C1.2, C2.2, IC1.4, IC2.4, R11.1, R25.2, R26.1, R46.2
Routing:
- net GND: track 959.3 -> 0.00 mm, vias 34 -> 0
- net BAT2-: track 478.5 -> 0.00 mm, vias 10 -> 0
- net 3.3: track 423.4 -> 0.00 mm, vias 17 -> 0
- net VIN_RAW: track 395.4 -> 0.00 mm, vias 15 -> 0
- net VUSB: track 294.5 -> 0.00 mm, vias 8 -> 0
- net N$28: track 272.1 -> 0.00 mm, vias 7 -> 0
- net IMU_SCL: track 229.1 -> 0.00 mm, vias 4 -> 0
- net IN2: track 185.0 -> 0.00 mm, vias 8 -> 0
- net N$30: track 168.9 -> 0.00 mm, vias 3 -> 0
- net BTN2: track 146.0 -> 0.00 mm, vias 1 -> 0
- net VCC: track 140.7 -> 0.00 mm, vias 7 -> 0
- net ADDR1: track 137.3 -> 0.00 mm, vias 9 -> 0
- net BTN3: track 134.6 -> 0.00 mm, vias 3 -> 0
- net OPTICAL_EN2: track 133.7 -> 0.00 mm, vias 10 -> 0
- net BTN4: track 130.5 -> 0.00 mm, vias 6 -> 0
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- removed copper zone on layer 1, net GND
- removed copper zone on layer 16, net GND

Commit message: Wip
Parts:
- removed C1, C12, C13, C14, C2, C3, C4, C7, C9: (no value), rcl:153CLV-1010
- removed D2: (no value), SparkFun-DiscreteSemi:SOD-323
- removed R28: 1.5K, SparkFun-Passives:0805
- removed R50: 10K, SparkFun-Passives:0805
- removed U$11: 220uF, rhoban:PANASONIC_D8
- removed U$2, U$4, U$5, U$6: CONNEC_1X01PAD, rhoban:1_PAD
- removed U$3, U$9: 47uF, rhoban:PANASONIC_D
- added C17, C18: 0.1uF, SparkFun-Passives:0805
- added C19, C20: 2200uF, rcl:E5-13
- added IC1: FT232L, rhoban:SSOP28
- added R10, R9: 10K, rcl:R0805
- added R11: 2K, rcl:R0805
- added R7: 470, rcl:R0805
- added U$7: S8252, rhoban:SOT23-6
- added U2: ESP32-WROOM-32E_(16MB), ESP32-WROOM-32E__16MB_:MODULE_ESP32-WROOM-32E_(16MB)
- added U3, U4: IRLMS2002TRPBF, rhoban:SOT23-6
- U$1: value CONNEC_1X01PAD -> KICKER; device rhoban:1_PAD -> rhoban:KICKER
- moved L1 240.7 mm to (107.4, -47.9)
- moved D1 240.7 mm to (129.4, -52.8)
- moved U1 240.7 mm to (141.9, -28.7)
- moved C15 240.7 mm to (104.4, -54.2)
- moved C16 240.7 mm to (110.1, -54.2)
- moved R1 240.7 mm to (106.0, -40.5)
- moved R2 240.7 mm to (120.3, -54.2)
- moved R4 240.7 mm to (115.8, -54.2)
- moved R6 219.3 mm to (-21.0, 22.6)
- moved U$1 214.8 mm to (-59.7, 25.8), turned to 330 degrees
- moved X20 189.3 mm to (32.4, 30.9), turned to 300 degrees
- moved MOS 182.2 mm to (-27.3, 29.3), turned to 60 degrees
- moved REG 143.1 mm to (5.59, 3.94)
- moved REG1 141.1 mm to (2.92, -5.08)
- moved U$13 25.7 mm to (0.89, -18.0)
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Connections:
- removed net BAT1+: U$14.P3
- removed net BAT2+: U$14.P5
- removed net BAT2-: U$14.P2
- removed net BAT2CHARGE: U$14.P4
- removed net DISC: R28.1, R50.2
- new net GND_RAW: C17.2, C18.1, R10.2, U$14.P4, U$7.6, U4.4, X20.3
- new net N$10: U3.1, U3.2, U3.5, U3.6, U4.1, U4.2, U4.5, U4.6
- new net N$11: U$7.2, U3.3
- new net N$12: U$7.1, U4.3
- new net N$13: R11.1, U$14.P5, U$7.3
- new net N$14: IC1.1, U2.35
- new net N$15: IC1.5, U2.34
- new net N$7: U$14.P2, X20.2
- new net N$8: R7.1, U$7.5
- new net N$9: C18.2, R10.1, R9.2, U$7.4
- net 3.3: no longer U$9.+
- net 3.3V: now also IC1.20, IC1.4, U2.2
- net BUZZER: now also U2.8
- net GND: now also C19.-, C20.-, IC1.18, IC1.21, IC1.25, IC1.7, R11.2, U2.1, U2.15, U2.38, U2.39_1, U2.39_10, U2.39_11, U2.39_12, U2.39_13, U2.39_14, U2.39_15, U2.39_16, U2.39_17, U2.39_18, U2.39_19, U2.39_2, U2.39_20, U2.39_21, U2.39_3, U2.39_4, U2.39_5, U2.39_6, U2.39_7, U2.39_8, U2.39_9, U3.4; no longer C1.-, C12.-, C13.-, C14.-, C2.-, C3.-, C4.-, C7.-, C9.-, R50.1, U$1.1, U$11.-, U$14.P1, U$3.-, U$9.-, X20.3
- net KICK: now also U2.9; no longer U$4.1
- net KICKER: now also U$1.2; no longer U$6.1
- net LEDS: now also U2.12
- net M1A: now also U2.16
- net M1B: now also U2.13
- net M1C1: now also U2.23
- net M1C2: now also U2.27
- net M2A: now also U2.28
- net M2B: now also U2.30
- net M2C1: now also U2.31
- net M2C2: now also U2.33
- net M3A: now also U2.36
- net M3B: now also U2.37
- net M3C1: now also U2.10
- net M3C2: now also U2.11
- net USBDM: now also IC1.16
- net USBDP: now also IC1.15; no longer R28.2
- net VCC: no longer U$3.+
- net VIN: now also R7.2, R9.1, U$14.P3; no longer D2.1, U$2.1, X20.2
- net VIN_RAW: no longer D2.2, U$11.+, U$14.P6
- net VSTORE: now also C19.+, C20.+, U$1.1; no longer C1.+, C12.+, C13.+, C14.+, C2.+, C3.+, C4.+, C7.+, C9.+, U$5.1
Other:
- board text removed: "3.3"
- board text removed: "IN1"
- board text removed: "IN2"
- board text removed: "RX1"
- board text removed: "SCL"
- board text removed: "SDA"
- board text removed: "TX"

Commit message: Wip
Parts:
- removed C17, C18: 0.1uF, SparkFun-Passives:0805
- removed CA4, CA5, CA6: C_EU-100NF, rhoban:C0805
- removed R29, R35: 22, SparkFun-Passives:0805
- removed R39: 1K, SparkFun-Passives:0805
- removed R40: 10K, SparkFun-Passives:0805
- removed RESET: KMR211GLFS, okie:PUSHBUTTON-KMR241GLFS
- added C1, C2, C3, C4, C7: 0.1µF, SparkFun-Capacitors:0805
- added R12, R13: 22, SparkFun-Resistors:0805
- C5, C6, C8: value 1uF -> 0.1µF; device SparkFun-Passives:0805 -> SparkFun-Capacitors:0805
- R1: device rcl:R2010 -> SparkFun-Resistors:0805
- R10, R11, R3, R5, R7, R9: device rcl:R0805 -> SparkFun-Resistors:0805
- R2, R4: device resistor:M0805 -> SparkFun-Resistors:0805
- R6: value (none) -> 0.3OHM-0805-1/8W-1%; device resistor:M0805 -> SparkFun-Resistors:0805
- moved D1 186.0 mm to (-46.9, 6.22), turned to 300 degrees
- moved U1 180.1 mm to (-35.4, 3.56), turned to 300 degrees
- moved R2 170.8 mm to (-39.0, 7.51), turned to 210 degrees
- moved R4 170.5 mm to (-42.8, 8.39), turned to 210 degrees
- moved C16 166.9 mm to (-43.2, 11.8), turned to 30 degrees
- moved R1 165.6 mm to (-50.8, 12.5), turned to 300 degrees
- moved L1 157.1 mm to (-42.1, 0.19), turned to 300 degrees
- moved C15 149.1 mm to (-32.2, 5.51), turned to 120 degrees
- moved C6 119.6 mm to (-0.13, 68.3), turned to 0 degrees
- moved R9 118.8 mm to (22.1, 22.4)
- moved R10 118.2 mm to (20.1, 17.1), turned to 270 degrees
- moved R11 116.6 mm to (28.8, 13.6), turned to 180 degrees
- moved R7 115.1 mm to (30.4, 21.2), turned to 90 degrees
- moved U3 112.2 mm to (23.1, 17.0)
- moved U4 111.8 mm to (26.8, 17.0)
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Connections:
- removed net N$6: R39.1, RESET.P$1, RESET.P$3
- removed net RESET: R40.2, RESET.P$2, RESET.P$4
- net 3.3: no longer R40.1
- net GND: now also C1.2, C2.2, C3.2, C4.2, C5.2, C6.2; no longer C5.1, C6.1, C8.1, CA4.2, CA5.2, CA6.2, R39.2
- net GND_RAW: now also C7.2, C8.1; no longer C17.2, C18.1
- net N$59: now also R12.1; no longer R29.1
- net N$60: now also R13.1; no longer R35.1
- net N$8: now also C8.2
- net N$9: now also C7.1; no longer C18.2
- net USBDM: now also R12.2; no longer R29.2
- net USBDP: now also R13.2; no longer R35.2
- net VCC: now also C4.1, C5.1, C6.1; no longer C5.2, C6.2, C8.2
- net VIN: now also R3.2
- net VIN_RAW: now also C1.1, C2.1, C3.1; no longer CA4.1, CA5.1, CA6.1, R3.2
- net VOLTAGE: now also U2.6
Other:
- board text added: "Junior-SSL rev0"
- board text removed: "Metabot Holo rev5"

Commit message: Rework done
Parts:
- removed U$1: KICKER, rhoban:KICKER
- removed X20: (no value), powersupply:DC-21MM
- added KICK_PADS: KICKER, rhoban:KICKER
- added U$10, U$11, U$15, U$2, U$3, U$4, U$5, U$6, U$8, U$9: (no value), SparkFun-Electromechanical:STAND-OFF
- added X2: (no value), powersupply:DC-21MM
- R8: device rcl:R0805 -> SparkFun-Resistors:0805
- moved U$14 4.45 mm to (35.7, 17.1)
- moved R11 4.16 mm to (25.3, 11.4)
- moved R5 4.16 mm to (21.4, 8.19)
- moved U$7 4.16 mm to (26.9, 14.9)
- moved U3 4.16 mm to (19.6, 14.9)
- moved U4 4.16 mm to (23.2, 14.9)
- moved C7 4.16 mm to (22.0, 19.2)
- moved R7 4.16 mm to (26.8, 19.1)
- moved R3 4.16 mm to (24.9, 8.24)
- moved C8 4.16 mm to (24.3, 19.1)
- moved R10 4.16 mm to (16.5, 15.0)
- moved R9 4.16 mm to (18.5, 20.2)
- moved C16 2.55 mm to (-45.7, 12.0)
- moved C20 2.47 mm to (-63.4, 17.4)
- moved C19 2.44 mm to (-46.4, 46.6)
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- renumbered JP1 to X1
Connections:
- net 1: now also X2.1; no longer X20.1
- net GND_RAW: now also X2.3; no longer X20.3
- net KICKER: now also KICK_PADS.2; no longer U$1.2
- net N$7: now also X2.2; no longer X20.2
- net VSTORE: now also KICK_PADS.1; no longer U$1.1
Other:
- board size 164.8 x 150.7 mm -> 170.3 x 155.9 mm
- board text removed: "VIN"
