File: electronics/holo/holo.sch (EAGLE design)
At the start: 92 parts, among them IC1 TP4056, IC2 TP4056, U1 CD4051BM, U2 CD4051BM, U4 CD4051BM

Commit message: Removing all components that will be replaced
Parts:
- removed BUT: KMR211GLFS, okie:BUTTON-KMR241GLFS
- removed C20, C21: 18pF, SparkFun-Passives:CAP0805
- removed CA2, CA3: C_EU-100NF, rhoban:C_EU-100NF
- removed D4, D5: Blue, SparkFun:LED1206
- removed EXT: CONNEC_1X09, rhoban:CONNEC_1X09
- removed IC1, IC2: TP4056, TP4056:TP4056
- removed OSC: 8MHz, SparkFun2:CRYSTAL5X3
- removed P1, P2: (no value), jst-ph:JST-PH2
- removed PROGRAM: CONNEC_1X066PADS, rhoban:CONNEC_1X066PADS
- removed R10, R12, R24, R9: 5K, SparkFun-Passives:RESISTOR0805-RES
- removed R11, R26, R30, R36, R46, R49: 1K, SparkFun-Passives:RESISTOR0805-RES
- removed R18, R48: 10K, SparkFun-Passives:RESISTOR0805-RES
- removed R25: 2K, SparkFun-Passives:RESISTOR0805-RES
- removed R37, R38: 10K, rcl:R-EU_R0805
- removed R47, R52: 4K, SparkFun-Passives:RESISTOR0805-RES
- removed U$10, U$7: (no value), rhoban:430186070716
- removed U$18: NPN_BC817,215, rhoban:NPN_BC817,215
- removed U$24: LM2940IMP-5.0, rhoban:LM2940IMP-5.0
- removed U$25: TS2940CW-3.3RP, rhoban:TS2940CW-3.3RP
- removed U$8: HOLO_OPTICALS, rhoban:HOLO_OPTICALS
- removed U2, U4: CD4051BM, rhoban:CD4051BM
- removed UC1: STM32F103CBT6, stm32:STM32F103CB
- added C13, C14, C9: (no value), rcl:CPOL-EU153CLV-1010
- added C15, C16: 22uF, resistor:C-EUC0805
- added L1: IHLP2525CZER220M11IND_IHLP_2525_CZ_VIS-M, INDUCTOR:IHLP2525CZER220M11IND_IHLP_2525_CZ_VIS-M
- added MOS: SUD50N04-8M8P-4GE3, rhoban:SUD50N04-8M8P-4GE3
- added R1: 270, rcl:R-EU_R2010
- added R2: 2k, resistor:R-EU_M0805
- added R4: 68k, resistor:R-EU_M0805
- added R6: (no value), resistor:R-EU_M0805
- added REG, REG1: REG_5V, rhoban:REG_5V
- added X20: DC21MMX, powersupply:DC21MMX
- C1, C2, C3, C4: value 10uF -> (none); device SparkFun-Passives:CAP0805 -> rcl:CPOL-EU153CLV-1010; FARNELL (none) -> 2610827
- C12, C7: value 1uF -> (none); device SparkFun-Passives:CAP0805 -> rcl:CPOL-EU153CLV-1010; FARNELL (none) -> 2610827
- D1: value Blue -> PMEG4030EP; device SparkFun:LED1206 -> nxp_60:PMEG4030EP; FARNELL 1581233 -> 1829201
- U$1: value GY-85 -> CONNEC_1X01PAD; device rhoban:GY-85 -> rhoban:CONNEC_1X01PAD; FARNELL 1593463 -> (none)
- U$2, U$6: value (none) -> CONNEC_1X01PAD; device rhoban:430186070716 -> rhoban:CONNEC_1X01PAD; FARNELL 2402407 -> (none)
- U$4: value HC05 -> CONNEC_1X01PAD; device rhoban:HC05 -> rhoban:CONNEC_1X01PAD; FARNELL MODULE HC-05 -> (none)
- U$5: value GP2 -> CONNEC_1X01PAD; device rhoban:GP2 -> rhoban:CONNEC_1X01PAD; FARNELL - -> (none)
- U1: value CD4051BM -> MT3608; device rhoban:CD4051BM -> MT3608:MT3608; FARNELL 2334931 -> (none)
Connections:
- removed net ADDR1: U1.A, U2.A, U4.A, UC1.PA15/JTDI
- removed net ADDR2: U1.B, U2.B, U4.B, UC1.PB4/NJTRST
- removed net ADDR3: U1.C, U2.C, U4.C, UC1.PA4/SPI1_NSS/USART2_CK/ADC12_IN4
- removed net A_INT: U$1.A_INT1
- removed net BOOT1: PROGRAM.4, UC1.PB2/BOOT1
- removed net BTN1: U$2.P$1, U2.4
- removed net BTN2: U$6.P$1, U4.4
- removed net BTN3: U$7.P$1, U1.5
- removed net BTN4: U$10.P$1, U2.5
- removed net BUTTON: BUT.2, BUT.4, R48.1, UC1.BOOT0, UC1.PA14/JTCK/SWCLK
- removed net CHARGE_EN: IC1.CE, IC2.CE, R25.1
- removed net G_DRDY: U$1.M_DRDY
- removed net G_INT: U$1.G_INT
- removed net HAS_USB: R46.1, UC1.PB12/SPI2_NSS/I2C2_SMBA/USART3_CK/TIM1_BKIN
- removed net IMU_NC: U$1.VCC_IN
- removed net IMU_SCL: EXT.7, U$1.SCL, UC1.PB10/I2C2_SCL/USART3_TX
- removed net IMU_SDA: EXT.6, U$1.SDA, UC1.PB11/I2C2_SDA/USART3_RX
- removed net IN1: EXT.8, U2.7
- removed net IN2: EXT.9, U4.7
- removed net KEY: UC1.PB8/TIM4_CH3
- removed net LED: R36.1, UC1.PA13/JTMS/SWDIO
- removed net MORE_CHARGE: R47.1, R52.1, UC1.PB14/SPI2_MISO/USART3_RTS/TIM1_CH2N
- removed net MRX: U$4.DOUT, UC1.PA3/USART2_RX/ADC12_IN3/TIM2_CH4
- removed net MTX: U$4.DIN, UC1.PA2/USART2_TX/ADC12_IN2/TIM2_CH3
- removed net MUX1: U1.COM_OUT/IN, UC1.PA1/USART2_RTS/ADC12_IN1/TIM2_CH2
- removed net MUX2: U2.COM_OUT/IN, UC1.PA5/SPI1_SCK/ADC12_IN5
- removed net MUX3: U4.COM_OUT/IN, UC1.PB1/ADC12_IN9/TIM3_CH4
- removed net N$20: D4.A, R26.2
- removed net N$21: D5.C, IC2.CHRG
- removed net N$22: IC2.STDBY, R12.1
- removed net N$23: D5.A, R11.2
- removed net N$26: BUT.1, BUT.3, R49.2
- removed net N$29: D1.A, R36.2
- removed net N$33: R30.2, U$18.B
- removed net N$8: IC1.STDBY, R10.1
- removed net OPTICAL1: U$8.OPTICAL1, U1.2
- removed net OPTICAL2: U$8.OPTICAL2, U2.2
- removed net OPTICAL3: U$8.OPTICAL3, U4.2
- removed net OPTICAL4: U$8.OPTICAL4, U1.3
- removed net OPTICAL5: U$8.OPTICAL5, U2.3
- removed net OPTICAL6: U$8.OPTICAL6, U4.3
- removed net OPTICAL7: U$8.OPTICAL7, U1.4
- removed net OPTICAL_EN1: U$8.EN1, UC1.PC13-TAMPER-RTC
- removed net OPTICAL_EN2: U$8.EN2, UC1.PC14-OSC32_IN
- removed net OPTICAL_EN3: UC1.PC15-OSC32_OUT
- removed net OSC_IN: C21.2, OSC.2, UC1.PD0-OSC_IN
- removed net OSC_OUT: C20.2, OSC.1, UC1.PD1-OSC_OUT
- removed net P1: U$5.VO, U1.6
- removed net P2: U2.6
- removed net P3: U4.6
- removed net PROG1: IC1.PROG, R12.2, R24.2, R47.2
- removed net PROG2: IC2.PROG, R10.2, R52.2, R9.2
- removed net P_EN: R30.1, UC1.PB5/I2C1_SMBA
- removed net P_GND: U$18.C, U$5.GND
- removed net RX1: EXT.4, PROGRAM.6, R18.2, UC1.PA10/USART1_RX/TIM1_CH3
- removed net TX1: EXT.5, PROGRAM.5, UC1.PA9/USART1_TX/TIM1_CH2
- removed net VOLTAGE1: R3.1, R5.2, U4.5
- removed net VOLTAGE2: R37.1, R38.2, U1.7
- removed net XBEECONF: U$4.KEY, UC1.PB3/JTDO
- new net 3.3V: REG1.OUT
- new net KICK: MOS.G, R6.1, U$4.1
- new net KICKER: MOS.D, U$6.1
- new net N$1: D1.A, L1.1, U1.SW
- new net N$4: R2.2, R4.1, U1.FB
- new net VOLTAGE: R3.1, R5.2
- new net VSTORE: C1.+, C12.+, C13.+, C14.+, C2.+, C3.+, C4.+, C7.+, C9.+, R1.1, U$5.1
- net 3.3: no longer C12.2, C7.2, CA3.1, EXT.2, PROGRAM.2, R49.1, U$1.3.3, U$25.OUT, U$4.3.3V, U$8.3.3V, U1.VDD, U2.VDD, U4.VDD, UC1.VDD_1, UC1.VDD_2, UC1.VDD_3, UC1.VDD_A
- net BAT1+: no longer C3.2, IC1.BAT, P2.2
- net BAT2+: no longer P1.2
- net BAT2-: no longer C5.2, C6.2, C8.2, LED1.VDD, LED2.VDD, LED3.VDD, LED4.VDD, LED5.VDD, LED6.VDD, P1.1, R37.2, U$8.VIN
- net BAT2CHARGE: no longer C4.2, IC2.BAT
- net BUZZER: no longer UC1.PA0_WKUP/USART2_CTS/ADC12_IN0/TIM2_CH1_ETR
- net DISC: no longer UC1.PB9/TIM4_CH4
- net GND: now also C1.-, C12.-, C13.-, C14.-, C15.2, C16.2, C2.-, C3.-, C4.-, C7.-, C9.-, MOS.S, R2.1, R6.2, REG.GND, REG1.GND, U$1.1, U1.GND, X20.3; no longer C1.1, C12.1, C2.1, C20.1, C21.1, C3.1, C4.1, C7.1, CA2.2, CA3.2, D1.C, EXT.1, IC1.GND, IC1.TEMP, IC2.GND, IC2.TEMP, P2.1, PROGRAM.1, R18.1, R24.1, R38.1, R48.2, R9.1, U$1.GND, U$10.P$2, U$18.E, U$2.P$2, U$24.GND, U$25.GND, U$4.GND, U$6.P$2, U$7.P$2, U$8.GND, U1.INH, U1.VEE, U1.VSS, U2.INH, U2.VEE, U2.VSS, U4.INH, U4.VEE, U4.VSS, UC1.VSS_1, UC1.VSS_2, UC1.VSS_3, UC1.VSS_A
- net LEDS: no longer UC1.PB15/SPI2_MOSI/TIM1_CH3N
- net M1A: no longer UC1.PB7/I2C1_SDA/TIM4_CH2
- net M1B: no longer UC1.PB6/I2C1_SCL/TIM4_CH1
- net M1C1: no longer U1.0
- net M1C2: no longer U2.0
- net M2A: no longer UC1.PA6/SPI1_MISO/ADC12_IN6/TIM3_CH1
- net M2B: no longer UC1.PA8/USART1_CK/TIM1_CH1/MCO
- net M2C1: no longer U4.0
- net M2C2: no longer U1.1
- net M3A: no longer UC1.PB0/ADC12_IN8/TIM3_CH3
- net M3B: no longer UC1.PA7/SPI1_MOSI/ADC12_IN7/TIM3_CH2
- net M3C1: no longer U2.1
- net M3C2: no longer U4.1
- net N$2: now also C16.1, D1.K, R1.2, R4.2; no longer D4.C, IC1.CHRG
- net RESET: no longer PROGRAM.3, UC1.NRST
- net USBDM: no longer UC1.PA11/USART1_CTS/CAN_RX/TIM1_CH4/USBDM
- net USBDP: no longer UC1.PA12/USART1_RTS/CAN_TX/TIM1_ETR/USBDP
- net VCC: now also C5.2, C6.2, C8.2, LED1.VDD, LED2.VDD, LED3.VDD, LED4.VDD, LED5.VDD, LED6.VDD, REG.OUT; no longer CA2.1, U$24.OUT, U$25.IN, U$5.VCC
- net VIN: now also C15.1, L1.2, REG.IN, REG1.IN, U$2.1, U1.EN, U1.IN, X20.2; no longer U$24.IN
- net VIN_RAW: no longer EXT.3
- net VUSB: no longer C1.2, C2.2, IC1.VCC, IC2.VCC, R11.1, R25.2, R26.1, R46.2
Other:
- note added: "TODO: Add kicker holes footprint"
- note added: "TODO: Connect kicker components"
- note added: "TODO: Handle VM initialization (DPDT?)"
- note added: "TODO: Handle power switch"
- note added: "TODO: Source ESP32 footprint"
- note added: "TODO: Source FTDI (see wroom schematic)"
- note added: "TODO: Source MOS for BMS"
- note removed: "BOOT0"
- note removed: "BT & IMU"
- note removed: "BUTTONS"
- note removed: "Blue"
- note removed: "GP2"
- note removed: "MULTIPLEXERS"
- note removed: "OPTICALS"
- note removed: "STM32"

Commit message: Wip
Parts:
- removed C1, C12, C13, C14, C2, C3, C4, C7, C9: (no value), rcl:CPOL-EU153CLV-1010
- removed D2: (no value), SparkFun-DiscreteSemi:DIODESOD
- removed R28: 1.5K, SparkFun-Passives:RESISTOR0805-RES
- removed R50: 10K, SparkFun-Passives:RESISTOR0805-RES
- removed U$11: 220uF, rhoban:CPOL_EUPANASONIC_D8
- removed U$2, U$4, U$5, U$6: CONNEC_1X01PAD, rhoban:CONNEC_1X01PAD
- removed U$3, U$9: 47uF, rhoban:CPOL_EUPANASONIC_D
- added C17, C18: 0.1uF, SparkFun-Passives:CAP0805
- added C19, C20: 2200uF, rcl:CPOL-EUE5-13
- added IC1: FT232L, rhoban:FT232L
- added R10, R9: 10K, rcl:R-EU_R0805
- added R11: 2K, rcl:R-EU_R0805
- added R7: 470, rcl:R-EU_R0805
- added U$7: S8252, rhoban:S8252
- added U2: ESP32-WROOM-32E_(16MB), ESP32-WROOM-32E__16MB_:ESP32-WROOM-32E_(16MB)
- added U3, U4: IRLMS2002TRPBF, rhoban:IRLMS2002TRPBF
- U$1: value CONNEC_1X01PAD -> KICKER; device rhoban:CONNEC_1X01PAD -> rhoban:KICKER
Connections:
- removed net BAT1+: U$14.P$4
- removed net BAT2+: U$14.P$2
- removed net BAT2-: U$14.P$1
- removed net BAT2CHARGE: U$14.P$5
- removed net DISC: R28.1, R50.2
- new net GND_RAW: C17.2, C18.1, R10.2, U$14.P$5, U$7.VSS, U4.S, X20.3
- new net N$10: U3.D, U4.D
- new net N$11: U$7.CO, U3.G
- new net N$12: U$7.DO, U4.G
- new net N$13: R11.1, U$14.P$2, U$7.VM
- new net N$14: IC1.TXD, U2.TXD0
- new net N$15: IC1.RXD, U2.RXD0
- new net N$7: U$14.P$1, X20.2
- new net N$8: R7.1, U$7.VDD
- new net N$9: C18.2, R10.1, R9.2, U$7.VC
- net 3.3: no longer U$9.+
- net 3.3V: now also IC1.VCC, IC1.VCCIO, U2.3V3
- net BUZZER: now also U2.IO32
- net GND: now also C19.-, C20.-, IC1.GND, IC1.GND@1, IC1.GND@2, IC1.GND@A, R11.2, U2.GND, U3.S; no longer C1.-, C12.-, C13.-, C14.-, C2.-, C3.-, C4.-, C7.-, C9.-, R50.1, U$1.1, U$11.-, U$14.P$3, U$3.-, U$9.-, X20.3
- net KICK: now also U2.IO33; no longer U$4.1
- net KICKER: now also U$1.2; no longer U$6.1
- net LEDS: now also U2.IO27
- net M1A: now also U2.IO13
- net M1B: now also U2.IO14
- net M1C1: now also U2.IO15
- net M1C2: now also U2.IO16
- net M2A: now also U2.IO17
- net M2B: now also U2.IO18
- net M2C1: now also U2.IO19
- net M2C2: now also U2.IO21
- net M3A: now also U2.IO22
- net M3B: now also U2.IO23
- net M3C1: now also U2.IO25
- net M3C2: now also U2.IO26
- net USBDM: now also IC1.USBDM
- net USBDP: now also IC1.USBDP; no longer R28.2
- net VCC: no longer U$3.+
- net VIN: now also R7.2, R9.1, U$14.P$4; no longer D2.C, U$2.1, X20.2
- net VIN_RAW: no longer D2.A, U$11.+, U$14.P$6
- net VSTORE: now also C19.+, C20.+, U$1.1; no longer C1.+, C12.+, C13.+, C14.+, C2.+, C3.+, C4.+, C7.+, C9.+, U$5.1
Other:
- note added: "RDS(on) is 30mohm. If BMS cut at 200mV, it is ~3.5A"
- note added: "TODO: Add spacers to protect the robot"
- note removed: "TODO: Connect kicker components"
- note removed: "TODO: Handle VM initialization (DPDT?)"
- note removed: "TODO: Source ESP32 footprint"
- note removed: "TODO: Source FTDI (see wroom schematic)"
- note removed: "TODO: Source MOS for BMS"
- moved on the sheet: D3, MOS, R3, R5, R6

Commit message: Wip
Parts:
- removed C17, C18: 0.1uF, SparkFun-Passives:CAP0805
- removed CA4, CA5, CA6: C_EU-100NF, rhoban:C_EU-100NF
- removed R29, R35: 22, SparkFun-Passives:RESISTOR0805-RES
- removed R39: 1K, SparkFun-Passives:RESISTOR0805-RES
- removed R40: 10K, SparkFun-Passives:RESISTOR0805-RES
- removed RESET: KMR211GLFS, okie:BUTTON-KMR241GLFS
- added C1, C2, C3, C4, C7: 0.1µF, SparkFun-Capacitors:0.33UF/330NF-0805-50V-10%
- added R12, R13: 22, SparkFun-Resistors:0.3OHM-0805-1/8W-1%
- C5, C6, C8: value 1uF -> 0.1µF; device SparkFun-Passives:CAP0805 -> SparkFun-Capacitors:0.33UF/330NF-0805-50V-10%; PROD_ID (none) -> CAP-08469; VALUE (none) -> 0.33µF
- R1: device rcl:R-EU_R2010 -> SparkFun-Resistors:0.3OHM-0805-1/8W-1%
- R10, R11, R3, R5, R7, R9: device rcl:R-EU_R0805 -> SparkFun-Resistors:0.3OHM-0805-1/8W-1%
- R2, R4: device resistor:R-EU_M0805 -> SparkFun-Resistors:0.3OHM-0805-1/8W-1%
- R6: value (none) -> 0.3OHM-0805-1/8W-1%; device resistor:R-EU_M0805 -> SparkFun-Resistors:0.3OHM-0805-1/8W-1%
Connections:
- removed net N$6: R39.1, RESET.1, RESET.3
- removed net RESET: R40.2, RESET.2, RESET.4
- net 3.3: no longer R40.1
- net GND: now also C1.2, C2.2, C3.2, C4.2, C5.2, C6.2; no longer C5.1, C6.1, C8.1, CA4.2, CA5.2, CA6.2, R39.2
- net GND_RAW: now also C7.2, C8.1; no longer C17.2, C18.1
- net N$59: now also R12.1; no longer R29.1
- net N$60: now also R13.1; no longer R35.1
- net N$8: now also C8.2
- net N$9: now also C7.1; no longer C18.2
- net USBDM: now also R12.2; no longer R29.2
- net USBDP: now also R13.2; no longer R35.2
- net VCC: now also C4.1, C5.1, C6.1; no longer C5.2, C6.2, C8.2
- net VIN: now also R3.2
- net VIN_RAW: now also C1.1, C2.1, C3.1; no longer CA4.1, CA5.1, CA6.1, R3.2
- net VOLTAGE: now also U2.IO34
Other:
- note removed: "TODO: Handle power switch"
- moved on the sheet: C5, C6

Commit message: Rework done
Parts:
- C1, C2, C3, C4, C5, C6, C7, C8: FARNELL (none) -> 2688486RL
- C10, C11: FARNELL (none) -> 1081223
- IC1: FARNELL (none) -> 1146032
- R10, R9: FARNELL (none) -> 2074334RL
- R11: FARNELL (none) -> 2447622
- R12, R13: FARNELL (none) -> 2446926
- R3: FARNELL (none) -> 2074395
- R5: FARNELL 2447553 -> 2074334RL
- R7: FARNELL (none) -> 2447662
- R8: device rcl:R-EU_R0805 -> SparkFun-Resistors:0.3OHM-0805-1/8W-1%; FARNELL (none) -> 2447622
- U$16, U$17, U$21: FARNELL JST-XH 6P -> 9491805
- U$7: FARNELL (none) -> https://www.digikey.fr/fr/products/detail/ablic-u-s-a-inc/S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; REF (none) -> S-8252AAL-M6T1U
- U1: FARNELL (none) -> MT3608
- U3, U4: FARNELL (none) -> 2577180RL
- X2: FARNELL (none) -> 1217037
- renumbered JP1 to X1, U$1 to KICK_PADS, X20 to X2
Other:
- note added: "BMS cut at 0.2V, so ~3.3A"
- note added: "RDSon is ~30 mohm. So "Rsense" is 60mohm"
- note removed: "RDS(on) is 30mohm. If BMS cut at 200mV, it is ~3.5A"
- note removed: "TODO: Add kicker holes footprint"
- note removed: "TODO: Add spacers to protect the robot"
- moved on the sheet: D3, R3, R5
